File: First pcb 65%.kicad_pcb (KiCad board)
At the start: 2 copper layers, 0 parts

Commit message: pcb updates
Parts:
- added C1: 22pF, Capacitor_SMD:C_0805_2012Metric, F.Cu at (215.7, 119.2)
- added C2: 22pF, Capacitor_SMD:C_0805_2012Metric, F.Cu at (207.0, 119.2)
- added C3: 1uF, Capacitor_SMD:C_0805_2012Metric, F.Cu at (201.9, 107.4)
- added C4: 0.1uF, Capacitor_SMD:C_0805_2012Metric, F.Cu at (224.4, 111.3)
- added C5: 0.1uF, Capacitor_SMD:C_0805_2012Metric, F.Cu at (220.8, 108.9)
- added C6: 0.1uF, Capacitor_SMD:C_0805_2012Metric, F.Cu at (220.4, 100.7)
- added C7: 10uF, Capacitor_SMD:C_0805_2012Metric, F.Cu at (226.4, 115.2)
- added D1: SOD-123, Diode_SMD:D_SOD-123, F.Cu at (69.3, 37.6)
- added D10: SOD-123, Diode_SMD:D_SOD-123, F.Cu at (240.7, 38.2)
- added D11: SOD-123, Diode_SMD:D_SOD-123, F.Cu at (259.8, 38.2)
- added D12: SOD-123, Diode_SMD:D_SOD-123, F.Cu at (278.8, 38.2)
- added D13: SOD-123, Diode_SMD:D_SOD-123, F.Cu at (297.8, 38.2)
- added D14: SOD-123, Diode_SMD:D_SOD-123, F.Cu at (322.8, 43.7)
- added D15: SOD-123, Diode_SMD:D_SOD-123, F.Cu at (352.4, 43.9)
- added D16: SOD-123, Diode_SMD:D_SOD-123, F.Cu at (74.0, 57.5)
- added D17: SOD-123, Diode_SMD:D_SOD-123, F.Cu at (97.8, 57.5)
- added D18: SOD-123, Diode_SMD:D_SOD-123, F.Cu at (116.9, 57.5)
- added D19: SOD-123, Diode_SMD:D_SOD-123, F.Cu at (135.9, 57.5)
- added D2: SOD-123, Diode_SMD:D_SOD-123, F.Cu at (88.2, 37.7)
- added D20: SOD-123, Diode_SMD:D_SOD-123, F.Cu at (154.9, 57.5)
- added D21: SOD-123, Diode_SMD:D_SOD-123, F.Cu at (174.0, 57.4)
- added D22: SOD-123, Diode_SMD:D_SOD-123, F.Cu at (193.1, 57.4)
- added D23: SOD-123, Diode_SMD:D_SOD-123, F.Cu at (212.1, 57.4)
- added D24: SOD-123, Diode_SMD:D_SOD-123, F.Cu at (231.2, 57.5)
- added D25: SOD-123, Diode_SMD:D_SOD-123, F.Cu at (250.2, 57.5)
- added D26: SOD-123, Diode_SMD:D_SOD-123, F.Cu at (269.3, 57.5)
- added D27: SOD-123, Diode_SMD:D_SOD-123, F.Cu at (288.3, 57.5)
- added D28: SOD-123, Diode_SMD:D_SOD-123, F.Cu at (307.4, 57.5)
- added D29: SOD-123, Diode_SMD:D_SOD-123, F.Cu at (330.7, 57.5)
- added D3: SOD-123, Diode_SMD:D_SOD-123, F.Cu at (107.4, 37.7)
- added D30: SOD-123, Diode_SMD:D_SOD-123, F.Cu at (351.6, 62.8)
- added D31: SOD-123, Diode_SMD:D_SOD-123, F.Cu at (48.5, 77.8)
- added D32: SOD-123, Diode_SMD:D_SOD-123, F.Cu at (75.9, 77.2)
- added D33: SOD-123, Diode_SMD:D_SOD-123, F.Cu at (102.6, 76.6)
- added D34: SOD-123, Diode_SMD:D_SOD-123, F.Cu at (121.6, 76.6)
- added D35: SOD-123, Diode_SMD:D_SOD-123, F.Cu at (140.7, 76.6)
- added D36: SOD-123, Diode_SMD:D_SOD-123, F.Cu at (159.7, 76.6)
- added D37: SOD-123, Diode_SMD:D_SOD-123, F.Cu at (178.8, 76.6)
- added D38: SOD-123, Diode_SMD:D_SOD-123, F.Cu at (197.8, 76.6)
- added D39: SOD-123, Diode_SMD:D_SOD-123, F.Cu at (216.9, 76.6)
- added D4: SOD-123, Diode_SMD:D_SOD-123, F.Cu at (126.4, 37.7)
- added D40: SOD-123, Diode_SMD:D_SOD-123, F.Cu at (236.0, 76.6)
- added D41: SOD-123, Diode_SMD:D_SOD-123, F.Cu at (255.0, 76.6)
- added D42: SOD-123, Diode_SMD:D_SOD-123, F.Cu at (274.1, 76.6)
- added D43: SOD-123, Diode_SMD:D_SOD-123, F.Cu at (293.1, 76.6)
- added D44: SOD-123, Diode_SMD:D_SOD-123, F.Cu at (321.4, 77.3)
- added D45: SOD-123, Diode_SMD:D_SOD-123, F.Cu at (351.4, 81.9)
- added D46: SOD-123, Diode_SMD:D_SOD-123, F.Cu at (45.4, 95.3)
- added D47: SOD-123, Diode_SMD:D_SOD-123, F.Cu at (77.5, 102.0)
- added D48: SOD-123, Diode_SMD:D_SOD-123, F.Cu at (112.1, 97.1)
- added D49: SOD-123, Diode_SMD:D_SOD-123, F.Cu at (131.2, 97.1)
- added D5: SOD-123, Diode_SMD:D_SOD-123, F.Cu at (145.4, 37.8)
- added D50: SOD-123, Diode_SMD:D_SOD-123, F.Cu at (150.2, 97.1)
- added D51: SOD-123, Diode_SMD:D_SOD-123, F.Cu at (169.3, 97.2)
- added D52: SOD-123, Diode_SMD:D_SOD-123, F.Cu at (188.3, 97.2)
- added D53: SOD-123, Diode_SMD:D_SOD-123, F.Cu at (207.4, 97.2)
- added D54: SOD-123, Diode_SMD:D_SOD-123, F.Cu at (226.4, 97.2)
- added D55: SOD-123, Diode_SMD:D_SOD-123, F.Cu at (245.5, 97.2)
- added D56: SOD-123, Diode_SMD:D_SOD-123, F.Cu at (264.5, 97.2)
- added D57: SOD-123, Diode_SMD:D_SOD-123, F.Cu at (283.6, 97.2)
- added D58: SOD-123, Diode_SMD:D_SOD-123, F.Cu at (309.3, 96.2)
- added D59: SOD-123, Diode_SMD:D_SOD-123, F.Cu at (335.9, 96.2)
- added D6: SOD-123, Diode_SMD:D_SOD-123, F.Cu at (164.5, 37.8)
- added D60: SOD-123, Diode_SMD:D_SOD-123, F.Cu at (351.5, 101.0)
- added D61: SOD-123, Diode_SMD:D_SOD-123, F.Cu at (45.4, 115.1)
- added D62: SOD-123, Diode_SMD:D_SOD-123, F.Cu at (71.6, 114.3)
- added D63: SOD-123, Diode_SMD:D_SOD-123, F.Cu at (95.4, 114.4)
- added D64: SOD-123, Diode_SMD:D_SOD-123, F.Cu at (119.2, 114.8)
- added D65: SOD-123, Diode_SMD:D_SOD-123, F.Cu at (190.6, 115.2)
- added D66: SOD-123, Diode_SMD:D_SOD-123, F.Cu at (262.1, 115.6)
- added D67: SOD-123, Diode_SMD:D_SOD-123, F.Cu at (285.9, 115.6)
- added D68: SOD-123, Diode_SMD:D_SOD-123, F.Cu at (316.9, 115.5)
- added D69: SOD-123, Diode_SMD:D_SOD-123, F.Cu at (336.0, 115.5)
- added D7: SOD-123, Diode_SMD:D_SOD-123, F.Cu at (183.5, 37.8)
- added D70: SOD-123, Diode_SMD:D_SOD-123, F.Cu at (351.4, 120.0)
- added D8: SOD-123, Diode_SMD:D_SOD-123, F.Cu at (202.6, 38.1)
- added D9: SOD-123, Diode_SMD:D_SOD-123, F.Cu at (221.7, 38.1)
- added F1: 500m, Fuse:Fuse_1206_3216Metric, F.Cu at (45.3, 40.3)
- added J1: Conn_01x04, SSD1306:128x64OLED, F.Cu at (37.7, 51.8)
- added MX1: MX-NoLED, MX_Only:MXOnly-1U-NoLED, F.Cu at (61.0, 35.6)
- added MX10: MX-NoLED, MX_Only:MXOnly-1U-NoLED, F.Cu at (232.4, 35.6)
- added MX11: MX-NoLED, MX_Only:MXOnly-1U-NoLED, F.Cu at (251.5, 35.6)
- added MX12: MX-NoLED, MX_Only:MXOnly-1U-NoLED, F.Cu at (270.5, 35.6)
- added MX13: MX-NoLED, MX_Only:MXOnly-1U-NoLED, F.Cu at (289.6, 35.6)
- added MX14: MX-NoLED, MX_Only:MXOnly-2U-NoLED, F.Cu at (318.1, 35.6)
- added MX15: MX-NoLED, MX_Only:MXOnly-1U-NoLED, F.Cu at (346.7, 35.6)
- added MX16: MX-NoLED, MX_Only:MXOnly-1.5U-NoLED, F.Cu at (65.7, 54.6)
- added MX17: MX-NoLED, MX_Only:MXOnly-1U-NoLED, F.Cu at (89.5, 54.6)
- added MX18: MX-NoLED, MX_Only:MXOnly-1U-NoLED, F.Cu at (108.6, 54.6)
- added MX19: MX-NoLED, MX_Only:MXOnly-1U-NoLED, F.Cu at (127.6, 54.6)
- added MX2: MX-NoLED, MX_Only:MXOnly-1U-NoLED, F.Cu at (80.0, 35.6)
- added MX20: MX-NoLED, MX_Only:MXOnly-1U-NoLED, F.Cu at (146.7, 54.6)
- added MX21: MX-NoLED, MX_Only:MXOnly-1U-NoLED, F.Cu at (165.7, 54.6)
- added MX22: MX-NoLED, MX_Only:MXOnly-1U-NoLED, F.Cu at (184.8, 54.6)
- added MX23: MX-NoLED, MX_Only:MXOnly-1U-NoLED, F.Cu at (203.8, 54.6)
- added MX24: MX-NoLED, MX_Only:MXOnly-1U-NoLED, F.Cu at (222.9, 54.6)
- added MX25: MX-NoLED, MX_Only:MXOnly-1U-NoLED, F.Cu at (241.9, 54.6)
- added MX26: MX-NoLED, MX_Only:MXOnly-1U-NoLED, F.Cu at (261.0, 54.6)
- added MX27: MX-NoLED, MX_Only:MXOnly-1U-NoLED, F.Cu at (280.0, 54.6)
- added MX28: MX-NoLED, MX_Only:MXOnly-1U-NoLED, F.Cu at (299.1, 54.6)
- added MX29: MX-NoLED, MX_Only:MXOnly-1.5U-NoLED, F.Cu at (322.9, 54.6)
- added MX3: MX-NoLED, MX_Only:MXOnly-1U-NoLED, F.Cu at (99.1, 35.6)
- added MX30: MX-NoLED, MX_Only:MXOnly-1U-NoLED, F.Cu at (346.7, 54.6)
- added MX31: MX-NoLED, MX_Only:MXOnly-1.75U-NoLED, F.Cu at (68.1, 73.7)
- added MX32: MX-NoLED, MX_Only:MXOnly-1U-NoLED, F.Cu at (94.4, 73.7)
- added MX33: MX-NoLED, MX_Only:MXOnly-1U-NoLED, F.Cu at (113.4, 73.7)
- added MX34: MX-NoLED, MX_Only:MXOnly-1U-NoLED, F.Cu at (132.5, 73.7)
- added MX35: MX-NoLED, MX_Only:MXOnly-1U-NoLED, F.Cu at (151.5, 73.7)
- added MX36: MX-NoLED, MX_Only:MXOnly-1U-NoLED, F.Cu at (170.6, 73.7)
- added MX37: MX-NoLED, MX_Only:MXOnly-1U-NoLED, F.Cu at (189.6, 73.7)
- added MX38: MX-NoLED, MX_Only:MXOnly-1U-NoLED, F.Cu at (208.7, 73.7)
- added MX39: MX-NoLED, MX_Only:MXOnly-1U-NoLED, F.Cu at (227.7, 73.7)
- added MX4: MX-NoLED, MX_Only:MXOnly-1U-NoLED, F.Cu at (118.1, 35.6)
- added MX40: MX-NoLED, MX_Only:MXOnly-1U-NoLED, F.Cu at (246.8, 73.7)
- added MX41: MX-NoLED, MX_Only:MXOnly-1U-NoLED, F.Cu at (265.8, 73.7)
- added MX42: MX-NoLED, MX_Only:MXOnly-1U-NoLED, F.Cu at (284.9, 73.7)
- added MX43: MX-NoLED, MX_Only:MXOnly-2.25U-NoLED, F.Cu at (315.8, 73.7)
- added MX44: MX-NoLED, MX_Only:MXOnly-1U-NoLED, F.Cu at (346.7, 73.7)
- added MX45: MX-NoLED, MX_Only:MXOnly-1U-NoLED, F.Cu at (37.1, 92.7)
- added MX46: MX-NoLED, MX_Only:MXOnly-2.25U-NoLED, F.Cu at (72.9, 92.7)
- added MX47: MX-NoLED, MX_Only:MXOnly-1U-NoLED, F.Cu at (103.9, 92.7)
- added MX48: MX-NoLED, MX_Only:MXOnly-1U-NoLED, F.Cu at (122.9, 92.7)
- added MX49: MX-NoLED, MX_Only:MXOnly-1U-NoLED, F.Cu at (142.0, 92.7)
- added MX5: MX-NoLED, MX_Only:MXOnly-1U-NoLED, F.Cu at (137.2, 35.6)
- added MX50: MX-NoLED, MX_Only:MXOnly-1U-NoLED, F.Cu at (161.0, 92.7)
- added MX51: MX-NoLED, MX_Only:MXOnly-1U-NoLED, F.Cu at (180.1, 92.7)
- added MX52: MX-NoLED, MX_Only:MXOnly-1U-NoLED, F.Cu at (199.1, 92.7)
- added MX53: MX-NoLED, MX_Only:MXOnly-1U-NoLED, F.Cu at (218.2, 92.7)
- added MX54: MX-NoLED, MX_Only:MXOnly-1U-NoLED, F.Cu at (237.2, 92.7)
- added MX55: MX-NoLED, MX_Only:MXOnly-1U-NoLED, F.Cu at (256.3, 92.7)
- added MX56: MX-NoLED, MX_Only:MXOnly-1U-NoLED, F.Cu at (275.3, 92.7)
- added MX57: MX-NoLED, MX_Only:MXOnly-1.75U-NoLED, F.Cu at (301.5, 92.7)
- added MX58: MX-NoLED, MX_Only:MXOnly-1U-NoLED, F.Cu at (327.7, 92.7)
- added MX59: MX-NoLED, MX_Only:MXOnly-1U-NoLED, F.Cu at (346.8, 92.7)
- added MX6: MX-NoLED, MX_Only:MXOnly-1U-NoLED, F.Cu at (156.2, 35.6)
- added MX60: MX-NoLED, MX_Only:MXOnly-1U-NoLED, F.Cu at (37.2, 111.8)
- added MX61: MX-NoLED, MX_Only:MXOnly-1.25U-NoLED, F.Cu at (63.4, 111.8)
- added MX62: MX-NoLED, MX_Only:MXOnly-1.25U-NoLED, F.Cu at (87.2, 111.8)
- added MX63: MX-NoLED, MX_Only:MXOnly-1.25U-NoLED, F.Cu at (111.0, 111.8)
- added MX64: MX-NoLED, MX_Only:MXOnly-6.25U-NoLED, F.Cu at (182.3, 111.8)
- added MX65: MX-NoLED, MX_Only:MXOnly-1.25U-NoLED, F.Cu at (253.7, 111.8)
- added MX66: MX-NoLED, MX_Only:MXOnly-1.25U-NoLED, F.Cu at (277.5, 111.8)
- added MX67: MX-NoLED, MX_Only:MXOnly-1U-NoLED, F.Cu at (308.7, 111.8)
- added MX68: MX-NoLED, MX_Only:MXOnly-1U-NoLED, F.Cu at (327.7, 111.8)
- added MX69: MX-NoLED, MX_Only:MXOnly-1U-NoLED, F.Cu at (346.8, 111.8)
- added MX7: MX-NoLED, MX_Only:MXOnly-1U-NoLED, F.Cu at (175.3, 35.6)
- added MX8: MX-NoLED, MX_Only:MXOnly-1U-NoLED, F.Cu at (194.3, 35.6)
- added MX9: MX-NoLED, MX_Only:MXOnly-1U-NoLED, F.Cu at (213.4, 35.6)
- added R1: 22, Resistor_SMD:R_0805_2012Metric, F.Cu at (42.7, 44.0)
- added R2: 10k, Resistor_SMD:R_0805_2012Metric, F.Cu at (201.0, 118.4)
- added R3: 22, Resistor_SMD:R_0805_2012Metric, F.Cu at (36.9, 43.5)
- added R4: 5.1k, Resistor_SMD:R_0805_2012Metric, F.Cu at (34.2, 38.9)
- added R5: 5.1k, Resistor_SMD:R_0805_2012Metric, F.Cu at (46.2, 35.7)
- added R6: 10k, Resistor_SMD:R_0805_2012Metric, F.Cu at (222.7, 104.6)
- added R6: 22, Resistor_SMD:R_0805_2012Metric, F.Cu at (196.3, 104.4)
- added SW1: SW_Push, random-keyboard-parts:SKQG-1155865, F.Cu at (197.8, 113.5)
- added SW2: Rotary_Encoder_Switch, Rotary_Encoder:RotaryEncoder_Alps_EC11E-Switch_Vertical_H20mm, F.Cu at (29.6, 71.1)
- added U1: PRTR5V0U2X, random-keyboard-parts:SOT143B, F.Cu at (40.0, 39.5)
- added U2: ATmega32U4-AU, Package_QFP:TQFP-44_10x10mm_P0.8mm, F.Cu at (211.8, 107.4)
- added USB1: HRO-TYPE-C-31-M-12, Type-C:HRO-TYPE-C-31-M-12-HandSoldering, F.Cu at (40.2, 24.6)
- added Y1: 16MHz, Crystal:Crystal_SMD_3225-4Pin_3.2x2.5mm, F.Cu at (211.3, 119.1)
Other:
- board outline added: 328.7 x 96.8 mm
- net class Default: trace_width 0.25 -> 0.254
- net class Power added: clearance 0.2, trace_width 0.381, via_dia 0.8, via_drill 0.4

Commit message: routing
Parts:
- removed the R6 at (196.3, 104.4)
- C1, C2, C3, C4, C5, C6, C7, D1, D10, D11, D12, D13, D14, D15, D16, D17, D18, D19, D2, D20, D21, D22, D23, D24, D25, D26, D27, D28, D29, D3, D30, D31, D32, D33, D34, D35, D36, D37, D38, D39, D4, D40, D41, D42, D43, D44, D45, D46, D47, D48, D49, D5, D50, D51, D52, D53, D54, D55, D56, D57, D58, D59, D6, D60, D61, D62, D63, D64, D65, D66, D67, D68, D69, D7, D70, D8, D9, F1, R1, R2, R3, R4, R5, R6, U1, U2, USB1, Y1: moved to B.Cu
- SW1: footprint random-keyboard-parts:SKQG-1155865 -> Button_Switch_SMD:SW_SPST_SKQG_WithStem; moved to B.Cu
- moved R3 172.8 mm to (195.1, 113.0)
- moved R1 168.2 mm to (195.1, 114.9), turned to 180 degrees
- moved J1 21.8 mm to (38.2, 73.7), turned to 0 degrees
- moved C7 21.5 mm to (205.4, 119.8), turned to 0 degrees
- moved Y1 18.2 mm to (215.3, 101.3)
- moved C2 18.2 mm to (211.9, 101.6), turned to 270 degrees
- moved C1 18.1 mm to (218.9, 101.3), turned to 90 degrees
- moved R2 16.7 mm to (206.1, 102.5)
- moved R5 14.7 mm to (31.6, 33.9), turned to 180 degrees
- moved R4 13.8 mm to (47.2, 34.3)
- moved C6 12.3 mm to (208.3, 103.1), turned to 270 degrees
- moved C5 12.3 mm to (214.8, 119.7), turned to 180 degrees
- moved R6 11.6 mm to (222.6, 116.3), turned to 270 degrees
- moved SW1 10.2 mm to (199.1, 103.4)
- moved F1 9.60 mm to (35.7, 41.0), turned to 90 degrees
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Connections:
- net Net-(R1-Pad2) renamed /DP
- net Net-(R3-Pad1) renamed /DN
- R6 pad 1: GND -> Net-(R6-Pad1)
- R6 pad 2: Net-(R6-Pad2) -> GND
- U2 pad 10: Net-(U2-Pad10) -> ROW2
- U2 pad 11: Net-(U2-Pad11) -> ROW1
- U2 pad 12: Net-(U2-Pad12) -> ROW0
- U2 pad 20: Net-(U2-Pad20) -> EncB
- U2 pad 21: EncB -> EncA
- U2 pad 22: EncA -> COL0
- U2 pad 25: EncSW -> COL8
- U2 pad 26: Net-(U2-Pad26) -> COL2
- U2 pad 27: Net-(U2-Pad27) -> COL3
- U2 pad 28: Net-(U2-Pad28) -> COL4
- U2 pad 29: Net-(U2-Pad29) -> COL5
- U2 pad 30: Net-(U2-Pad30) -> COL6
- U2 pad 31: Net-(U2-Pad31) -> COL7
- U2 pad 32: Net-(U2-Pad32) -> COL1
- U2 pad 33: Net-(R6-Pad2) -> Net-(R6-Pad1)
- U2 pad 36: Net-(U2-Pad36) -> COL9
- U2 pad 37: Net-(U2-Pad37) -> COL10
- U2 pad 38: Net-(U2-Pad38) -> COL11
- U2 pad 39: Net-(U2-Pad39) -> COL12
- U2 pad 40: Net-(U2-Pad40) -> COL13
- U2 pad 41: Net-(U2-Pad41) -> COL14
- U2 pad 8: Net-(U2-Pad8) -> ROW4
- U2 pad 9: Net-(U2-Pad9) -> ROW3
Routing:
- net ROW1: track 0.00 -> 837.9 mm, vias 0 -> 22
- net COL7: track 0.00 -> 722.1 mm, vias 0 -> 19
- net ROW0: track 0.00 -> 714.0 mm, vias 0 -> 31
- net COL6: track 0.00 -> 665.5 mm, vias 0 -> 18
- net COL5: track 0.00 -> 627.8 mm, vias 0 -> 14
- net COL4: track 0.00 -> 557.2 mm, vias 0 -> 12
- net ROW2: track 0.00 -> 540.3 mm, vias 0 -> 18
- net COL3: track 0.00 -> 535.4 mm, vias 0 -> 15
- net COL8: track 0.00 -> 495.4 mm, vias 0 -> 11
- net COL2: track 0.00 -> 467.2 mm, vias 0 -> 19
- net GND: track 0.00 -> 431.7 mm, vias 0 -> 15
- net COL9: track 0.00 -> 405.0 mm, vias 0 -> 15
- net ROW3: track 0.00 -> 402.2 mm, vias 0 -> 28
- net COL1: track 0.00 -> 397.1 mm, vias 0 -> 19
- net COL12: track 0.00 -> 387.4 mm, vias 0 -> 3
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- added copper zone on B.Cu, net GND
- added copper zone on F.Cu, net GND
Other:
- board size 328.7 x 96.8 mm -> 328.7 x 97.9 mm
