File: First pcb 65%.sch (KiCad schematic (older format))
At the start: 18 parts

Commit message: added plate file and pcb progress
Parts:
- added D? (x3): SOD-123, symbol Device:D_Small
- added J?: Conn_01x04, symbol Connector_Generic:Conn_01x04
- added MX? (x3): MX-NoLED, symbol MX_Alps_Hybrid:MX-NoLED
- added SW?: Rotary_Encoder_Switch, symbol Device:Rotary_Encoder_Switch
Connections:
- net labels added: EncA, EncB, EncSW, SCL, SDA
- wire segments 59 -> 71
Other:
- moved on the sheet: C?, D?, F?, MX?, R?, SW?, U?, USB?, Y?

Commit message: more libraries
Parts:
- removed D? (x3): SOD-123, symbol Device:D_Small
- removed MX? (x3): MX-NoLED, symbol MX_Alps_Hybrid:MX-NoLED
- added D? (x68): SOD-123, symbol Device:D_Small
- added MX10, MX11, MX12, MX13, MX14, MX15, MX16, MX17, MX18, MX19, MX2, MX20, MX21, MX22, MX23, MX24, MX25, MX26, MX27, MX28, MX29, MX30, MX31, MX32, MX33, MX34, MX35, MX36, MX37, MX39, MX40, MX41, MX42, MX43, MX44, MX45, MX46, MX47, MX48, MX49, MX5, MX50, MX51, MX52, MX53, MX54, MX55, MX56, MX57, MX58, MX59, MX6, MX60, MX61, MX62, MX63, MX64, MX65, MX66, MX67, MX68, MX69, MX7, MX70, MX71, MX8, MX9: MX-NoLED, symbol MX_Alps_Hybrid:MX-NoLED
- added SW4: SW_Push, symbol Switch:SW_Push
- gave numbers to parts that had none: 3
Connections:
- net labels added: COL0, COL1, COL10, COL11, COL12, COL13, COL14, COL2, COL3, COL4, COL5, COL6, COL7, COL8, COL9, ROW0, ROW1, ROW2, ROW3, ROW4
- wire segments 71 -> 293
Other:
- moved on the sheet: C?, D?, F?, J?, MX1, R?, SW1, SW3, U?, USB?, Y?

Commit message: https://github.com/keebio/Keebio-Parts.pretty
Parts:
- removed F?: 500mA, symbol Device:Polyfuse_Small
- removed USB?: Molex-0548190589, symbol random-keyboard-parts:Molex-0548190589
- added D70: SOD-123, Diode_SMD:D_SOD-123, symbol Device:D_Small
- added F1: 500m, Fuse:Fuse_1206_3216Metric, symbol Device:Polyfuse_Small
- added MX60: MX-NoLED, MX_Only:MXOnly-1U-NoLED, symbol MX_Alps_Hybrid:MX-NoLED
- added R1, R3: 22, Resistor_SMD:R_0805_2012Metric, symbol Device:R_Small
- added R4, R5: 5.1k, Resistor_SMD:R_0805_2012Metric, symbol Device:R_Small
- added U1: PRTR5V0U2X, random-keyboard-parts:SOT143B, symbol random-keyboard-parts:PRTR5V0U2X
- added USB1: HRO-TYPE-C-31-M-12, Type-C:HRO-TYPE-C-31-M-12-HandSoldering, symbol Type-C:HRO-TYPE-C-31-M-12
- C1, C2, C3, C4, C5, C6, C7: renamed from C?; footprint (none) -> Capacitor_SMD:C_0805_2012Metric
- D1, D10, D11, D12, D13, D14, D15, D16, D17, D18, D19, D2, D20, D21, D22, D23, D24, D25, D26, D27, D28, D29, D3, D30, D31, D32, D33, D34, D35, D36, D37, D38, D39, D4, D40, D41, D42, D43, D44, D45, D46, D47, D48, D49, D5, D50, D51, D52, D53, D54, D55, D56, D57, D58, D59, D6, D60, D61, D62, D63, D64, D65, D66, D67, D68, D69, D7, D8, D9: renamed from D?; footprint (none) -> Diode_SMD:D_SOD-123
- MX1: footprint (none) -> MX_Only:MXOnly-1U-NoLED
- MX10: renamed from MX43; footprint (none) -> MX_Only:MXOnly-1U-NoLED
- MX11: renamed from MX47; footprint (none) -> MX_Only:MXOnly-1U-NoLED
- MX12: renamed from MX52; footprint (none) -> MX_Only:MXOnly-1U-NoLED
- MX13: renamed from MX57; footprint (none) -> MX_Only:MXOnly-1U-NoLED
- MX14: renamed from MX62; footprint (none) -> MX_Only:MXOnly-2U-NoLED
- MX15: renamed from MX67; footprint (none) -> MX_Only:MXOnly-1U-NoLED
- MX16: renamed from MX2; footprint (none) -> MX_Only:MXOnly-1.5U-NoLED
- MX17: renamed from MX8; footprint (none) -> MX_Only:MXOnly-1U-NoLED
- MX18: renamed from MX12; footprint (none) -> MX_Only:MXOnly-1U-NoLED
- MX19: renamed from MX17; footprint (none) -> MX_Only:MXOnly-1U-NoLED
- MX2: renamed from MX7; footprint (none) -> MX_Only:MXOnly-1U-NoLED
- MX20: renamed from MX22; footprint (none) -> MX_Only:MXOnly-1U-NoLED
- MX21: renamed from MX26; footprint (none) -> MX_Only:MXOnly-1U-NoLED
- MX22: renamed from MX30; footprint (none) -> MX_Only:MXOnly-1U-NoLED
- MX23: renamed from MX35; footprint (none) -> MX_Only:MXOnly-1U-NoLED
- MX24: renamed from MX40; footprint (none) -> MX_Only:MXOnly-1U-NoLED
- MX25: renamed from MX44; footprint (none) -> MX_Only:MXOnly-1U-NoLED
- MX26: renamed from MX48; footprint (none) -> MX_Only:MXOnly-1U-NoLED
- MX27: renamed from MX53; footprint (none) -> MX_Only:MXOnly-1U-NoLED
- MX28: renamed from MX58; footprint (none) -> MX_Only:MXOnly-1U-NoLED
- MX29: renamed from MX63; footprint (none) -> MX_Only:MXOnly-1.5U-NoLED
- MX3: renamed from MX11; footprint (none) -> MX_Only:MXOnly-1U-NoLED
- MX30: renamed from MX68; footprint (none) -> MX_Only:MXOnly-1U-NoLED
- MX31: renamed from MX9; footprint (none) -> MX_Only:MXOnly-1.75U-NoLED
- MX32: renamed from MX13; footprint (none) -> MX_Only:MXOnly-1U-NoLED
- MX33: renamed from MX18; footprint (none) -> MX_Only:MXOnly-1U-NoLED
- MX34: renamed from MX23; footprint (none) -> MX_Only:MXOnly-1U-NoLED
- MX35: renamed from MX27; footprint (none) -> MX_Only:MXOnly-1U-NoLED
- MX36: renamed from MX31; footprint (none) -> MX_Only:MXOnly-1U-NoLED
- MX37: renamed from MX36; footprint (none) -> MX_Only:MXOnly-1U-NoLED
- MX38: renamed from MX41; footprint (none) -> MX_Only:MXOnly-1U-NoLED
- MX39: renamed from MX45; footprint (none) -> MX_Only:MXOnly-1U-NoLED
- MX4: renamed from MX16; footprint (none) -> MX_Only:MXOnly-1U-NoLED
- MX40: renamed from MX49; footprint (none) -> MX_Only:MXOnly-1U-NoLED
- MX41: renamed from MX54; footprint (none) -> MX_Only:MXOnly-1U-NoLED
- MX42: renamed from MX59; footprint (none) -> MX_Only:MXOnly-1U-NoLED
- MX43: renamed from MX64; footprint (none) -> MX_Only:MXOnly-2.25U-NoLED
- MX44: renamed from MX69; footprint (none) -> MX_Only:MXOnly-1U-NoLED
- MX45: renamed from MX5; footprint (none) -> MX_Only:MXOnly-1U-NoLED
- MX46: renamed from MX10; footprint (none) -> MX_Only:MXOnly-2.25U-NoLED
- MX47: renamed from MX14; footprint (none) -> MX_Only:MXOnly-1U-NoLED
- MX48: renamed from MX19; footprint (none) -> MX_Only:MXOnly-1U-NoLED
- MX49: renamed from MX24; footprint (none) -> MX_Only:MXOnly-1U-NoLED
- MX5: renamed from MX21; footprint (none) -> MX_Only:MXOnly-1U-NoLED
- MX50: renamed from MX28; footprint (none) -> MX_Only:MXOnly-1U-NoLED
- MX51: renamed from MX32; footprint (none) -> MX_Only:MXOnly-1U-NoLED
- MX52: renamed from MX37; footprint (none) -> MX_Only:MXOnly-1U-NoLED
- MX53: renamed from MX42; footprint (none) -> MX_Only:MXOnly-1U-NoLED
- MX54: renamed from MX46; footprint (none) -> MX_Only:MXOnly-1U-NoLED
- MX55: renamed from MX50; footprint (none) -> MX_Only:MXOnly-1U-NoLED
- MX56: renamed from MX55; footprint (none) -> MX_Only:MXOnly-1U-NoLED
- MX57: renamed from MX60; footprint (none) -> MX_Only:MXOnly-1.75U-NoLED
- MX58: renamed from MX65; footprint (none) -> MX_Only:MXOnly-1U-NoLED
- MX59: renamed from MX70; footprint (none) -> MX_Only:MXOnly-1U-NoLED
- MX6: renamed from MX25; footprint (none) -> MX_Only:MXOnly-1U-NoLED
- MX61: renamed from MX6; footprint (none) -> MX_Only:MXOnly-1.25U-NoLED
- MX62: renamed from MX15; footprint (none) -> MX_Only:MXOnly-1.25U-NoLED
- MX63: renamed from MX20; footprint (none) -> MX_Only:MXOnly-1.25U-NoLED
- MX64: renamed from MX33; footprint (none) -> MX_Only:MXOnly-6.25U-NoLED
- MX65: renamed from MX51; footprint (none) -> MX_Only:MXOnly-1.25U-NoLED
- MX66: renamed from MX56; footprint (none) -> MX_Only:MXOnly-1.25U-NoLED
- MX67: renamed from MX61; footprint (none) -> MX_Only:MXOnly-1U-NoLED
- MX68: renamed from MX66; footprint (none) -> MX_Only:MXOnly-1U-NoLED
- MX69: renamed from MX71; footprint (none) -> MX_Only:MXOnly-1U-NoLED
- MX7: renamed from MX29; footprint (none) -> MX_Only:MXOnly-1U-NoLED
- MX8: renamed from MX34; footprint (none) -> MX_Only:MXOnly-1U-NoLED
- MX9: renamed from MX39; footprint (none) -> MX_Only:MXOnly-1U-NoLED
- R2, R6, R7, R8: renamed from R?; footprint (none) -> Resistor_SMD:R_0805_2012Metric
- SW1: footprint (none) -> random-keyboard-parts:SKQG-1155865
- SW2: renamed from SW3; footprint (none) -> Rotary_Encoder:RotaryEncoder_Alps_EC11E-Switch_Vertical_H20mm
- SW3: renamed from SW4; footprint (none) -> MX_Only:MXOnly-1U-NoLED
- Y1: renamed from Y?; footprint (none) -> Crystal:Crystal_SMD_3225-4Pin_3.2x2.5mm
- gave numbers to parts that had none: 2
Connections:
- net +5V: now also F1.1
- net COL0: now also MX60.1 (COL); no longer MX61.1 (COL)
- net COL1: now also MX61.1 (COL)
- net D+: now also R3.2
- net D-: now also R1.1
- net GND: now also R4.2, R5.2, U1.1 (GND), USB1.1 (GND), USB1.12 (GND), USB1.13 (SHIELD)
- net ROW4: now also D70.1 (K); no longer D64.1 (K)
- net VCC: now also F1.2, U1.4 (VCC), USB1.11 (VBUS), USB1.2 (VBUS)
- new net: R4.1, USB1.10 (CC2)
- new net: R5.1, USB1.4 (CC1)
- new net: R1.2, U1.3 (IO2), USB1.5 (DN2), USB1.7 (DN1)
- new net: R3.1, U1.2 (IO1), USB1.6 (DP1), USB1.8 (DP2)
- new net: D70.2 (A), MX60.2 (ROW)
- no-connect marks 0 -> 2
Other:
- moved on the sheet: D62, D63, D64, J1, MX61, MX62, MX63

Commit message: added i2c library and added footprints
Parts:
- J1: footprint (none) -> SSD1306:128x64OLED
Changed lines of the file:
@@
 F 0 "J1" H 13530 1592 50  0000 L CNN
 F 1 "Conn_01x04" H 13530 1501 50  0000 L CNN
-F 2 "" H 13450 1600 50  0001 C CNN
+F 2 "SSD1306:128x64OLED" H 13450 1600 50  0001 C CNN
 F 3 "~" H 13450 1600 50  0001 C CNN
 	1    13450 1600

Commit message: pcb updates
Parts:
- removed R6, R7: 22, Resistor_SMD:R_0805_2012Metric, symbol Device:R_Small
- removed SW3: SW_Push, MX_Only:MXOnly-1U-NoLED, symbol Switch:SW_Push
- renumbered D70 to D61, D61 to D65, D65 to D66, D66 to D67, D67 to D68, D68 to D69, D69 to D70, R8 to R6
Connections:
- net D+: now also U2.4 (D+)
- net D-: now also U2.3 (D-)
- net ROW4: now also D64.1 (K), D65.1 (K)
Other:
- moved on the sheet: D64, D65, MX63, MX64
Changed lines of the file:
@@
 	15650 4950 15750 4950
 $Comp
-L Device:R_Small R8
+L Device:R_Small R6
 U 1 1 614622D1
 P 15550 4950
-F 0 "R8" V 15354 4950 50  0000 C CNN
+F 0 "R6" V 15354 4950 50  0000 C CNN
 F 1 "10k" V 15445 4950 50  0000 C CNN
 F 2 "Resistor_SMD:R_0805_2012Metric" H 15550 4950 50  0001 C CNN
@@
 	0    1    1    0
 $EndComp
-$Comp
-L Device:R_Small R6
-U 1 1 61469FEB
-P 13900 3850
-F 0 "R6" V 13704 3850 50  0000 C CNN
-F 1 "22" V 13795 3850 50  0000 C CNN
-F 2 "Resistor_SMD:R_0805_2012Metric" H 13900 3850 50  0001 C CNN
-F 3 "~" H 13900 3850 50  0001 C CNN
-	1    13900 3850
-	0    1    1    0
-$EndComp
-$Comp
-L Device:R_Small R7
-U 1 1 6146ED31
-P 13600 4150
-F 0 "R7" V 13404 4150 50  0000 C CNN
-F 1 "22" V 13495 4150 50  0000 C CNN
-F 2 "Resistor_SMD:R_0805_2012Metric" H 13600 4150 50  0001 C CNN
-F 3 "~" H 13600 4150 50  0001 C CNN
-	1    13600 4150
-	0    1    1    0
-$EndComp
-Wire Wire Line
-	13800 3850 13650 3850
-Wire Wire Line
-	13500 4150 13400 4150
 $Comp
 L Device:C_Small C3
@@
 Wire Wire Line
 	14100 4150 13750 4150
-Wire Wire Line
-	14100 3850 14000 3850
 Wire Wire Line
 	15300 4950 15450 4950
@@
 $EndComp
 $Comp
-L Device:D_Small D67
+L Device:D_Small D68
 U 1 1 6155CB07
 P 8800 5800
-F 0 "D67" V 8846 5730 50  0000 R CNN
+F 0 "D68" V 8846 5730 50  0000 R CNN
 F 1 "SOD-123" V 8755 5730 50  0000 R CNN
 F 2 "Diode_SMD:D_SOD-123" V 8800 5800 50  0001 C CNN
@@
 $EndComp
 $Comp
-L Device:D_Small D68
+L Device:D_Small D69
 U 1 1 6155CB1C
 P 9300 5800
-F 0 "D68" V 9346 5730 50  0000 R CNN
+F 0 "D69" V 9346 5730 50  0000 R CNN
 F 1 "SOD-123" V 9255 5730 50  0000 R CNN
 F 2 "Diode_SMD:D_SOD-123" V 9300 5800 50  0001 C CNN
@@
 $EndComp
 $Comp
-L Device:D_Small D69
+L Device:D_Small D70
 U 1 1 6155CB31
 P 9800 5800
-F 0 "D69" V 9846 5730 50  0000 R CNN
+F 0 "D70" V 9846 5730 50  0000 R CNN
 F 1 "SOD-123" V 9755 5730 50  0000 R CNN
 F 2 "Diode_SMD:D_SOD-123" V 9800 5800 50  0001 C CNN
@@
 	8150 5700 8050 5700
 $Comp
-L Device:D_Small D66
+L Device:D_Small D67
 U 1 1 61572F78
 P 8050 5800
-F 0 "D66" V 8096 5730 50  0000 R CNN
+F 0 "D67" V 8096 5730 50  0000 R CNN
 F 1 "SOD-123" V 8005 5730 50  0000 R CNN
 F 2 "Diode_SMD:D_SOD-123" V 8050 5800 50  0001 C CNN
@@
 $EndComp
 $Comp
-L Device:D_Small D65
+L Device:D_Small D66
 U 1 1 61572F6E
 P 7400 5800
-F 0 "D65" V 7446 5730 50  0000 R CNN
+F 0 "D66" V 7446 5730 50  0000 R CNN
 F 1 "SOD-123" V 7355 5730 50  0000 R CNN
 F 2 "Diode_SMD:D_SOD-123" V 7400 5800 50  0001 C CNN
@@
 $EndComp
 Wire Wire Line
-	2950 4150 3100 4150
-Wire Wire Line
 	3150 4350 3150 4500
 Wire Wire Line
@@
 	6150 4100 6150 4800
 Connection ~ 6150 4800
-Wire Wire Line
-	6150 4800 6150 5450
-Wire Wire Line
-	6150 5450 6100 5450
-$Comp
-L Device:D_Small D61
+$Comp
+L Device:D_Small D65
 U 1 1 615AAD90
-P 5850 5750
-F 0 "D61" V 5896 5680 50  0000 R CNN
-F 1 "SOD-123" V 5805 5680 50  0000 R CNN
-F 2 "Diode_SMD:D_SOD-123" V 5850 5750 50  0001 C CNN
-F 3 "~" V 5850 5750 50  0001 C CNN
-	1    5850 5750
-	0    -1   -1   0
-$EndComp
-Wire Wire Line
-	5950 5650 5850 5650
+P 5850 5800
+F 0 "D65" V 5896 5730 50  0000 R CNN
+F 1 "SOD-123" V 5805 5730 50  0000 R CNN
+F 2 "Diode_SMD:D_SOD-123" V 5850 5800 50  0001 C CNN
+F 3 "~" V 5850 5800 50  0001 C CNN
+	1    5850 5800
+	0    -1   -1   0
+$EndComp
+Wire Wire Line
+	5950 5700 5850 5700
 $Comp
 L MX_Alps_Hybrid:MX-NoLED MX64
 U 1 1 615AAD85
-P 6000 5500
-F 0 "MX64" H 6033 5723 60  0000 C CNN
-F 1 "MX-NoLED" H 6033 5649 20  0000 C CNN
-F 2 "MX_Only:MXOnly-6.25U-NoLED" H 5375 5475 60  0001 C CNN
-F 3 "" H 5375 5475 60  0001 C CNN
-	1    6000 5500
-	1    0    0    -1
-$EndComp
-Connection ~ 6150 5450
+P 6000 5550
+F 0 "MX64" H 6033 5773 60  0000 C CNN
+F 1 "MX-NoLED" H 6033 5699 20  0000 C CNN
+F 2 "MX_Only:MXOnly-6.25U-NoLED" H 5375 5525 60  0001 C CNN
+F 3 "" H 5375 5525 60  0001 C CNN
+	1    6000 5550
+	1    0    0    -1
+$EndComp
 Wire Wire Line
 	5650 4800 5650 4100
@@
 	3250 4800 3150 4800
 Connection ~ 3250 4550
-$Comp
-L Switch:SW_Push SW3
-U 1 1 618DB5BA
-P 2450 4850
-F 0 "SW3" H 2450 5135 50  0000 C CNN
-F 1 "SW_Push" H 2450 5044 50  0000 C CNN
-F 2 "MX_Only:MXOnly-1U-NoLED" H 2450 5050 50  0001 C CNN
-F 3 "~" H 2450 5050 50  0001 C CNN
-	1    2450 4850
-	1    0    0    -1
-$EndComp
-Wire Wire Line
-	3050 4350 3050 4500
-Wire Wire Line
-	3050 4500 2600 4500
-Wire Wire Line
-	2600 4500 2600 4600
-Wire Wire Line
-	2600 4600 2750 4600
-Wire Wire Line
-	2750 4600 2750 4850
-Wire Wire Line
-	2750 4850 2650 4850
-Connection ~ 3050 4500
-Wire Wire Line
-	3050 4500 3050 4550
-Wire Wire Line
-	3100 4150 3100 3850
-Wire Wire Line
-	3100 3850 1950 3850
-Wire Wire Line
-	1950 3850 1950 4500
-Wire Wire Line
-	1950 4500 2250 4500
-Wire Wire Line
-	2250 4500 2250 4850
-Connection ~ 3100 4150
-Wire Wire Line
-	3100 4150 3150 4150
 Text GLabel 2500 3100 0    50   Input ~ 0
 ROW0
@@
 L Device:D_Small D64
 U 1 1 615A207D
-P 4350 5750
-F 0 "D64" V 4396 5680 50  0000 R CNN
-F 1 "SOD-123" V 4305 5680 50  0000 R CNN
-F 2 "Diode_SMD:D_SOD-123" V 4350 5750 50  0001 C CNN
-F 3 "~" V 4350 5750 50  0001 C CNN
-	1    4350 5750
-	0    -1   -1   0
-$EndComp
-Wire Wire Line
-	4450 5650 4350 5650
+P 4350 5800
+F 0 "D64" V 4396 5730 50  0000 R CNN
+F 1 "SOD-123" V 4305 5730 50  0000 R CNN
+F 2 "Diode_SMD:D_SOD-123" V 4350 5800 50  0001 C CNN
+F 3 "~" V 4350 5800 50  0001 C CNN
+	1    4350 5800
+	0    -1   -1   0
+$EndComp
+Wire Wire Line
+	4450 5700 4350 5700
 $Comp
 L MX_Alps_Hybrid:MX-NoLED MX63
 U 1 1 615A2062
-P 4500 5500
-F 0 "MX63" H 4533 5723 60  0000 C CNN
-F 1 "MX-NoLED" H 4533 5649 20  0000 C CNN
-F 2 "MX_Only:MXOnly-1.25U-NoLED" H 3875 5475 60  0001 C CNN
-F 3 "" H 3875 5475 60  0001 C CNN
-	1    4500 5500
+P 4500 5550
+F 0 "MX63" H 4533 5773 60  0000 C CNN
+F 1 "MX-NoLED" H 4533 5699 20  0000 C CNN
+F 2 "MX_Only:MXOnly-1.25U-NoLED" H 3875 5525 60  0001 C CNN
+F 3 "" H 3875 5525 60  0001 C CNN
+	1    4500 5550
 	1    0    0    -1
 $EndComp
@@
 	2800 5900 3350 5900
 $Comp
-L Device:D_Small D70
+L Device:D_Small D61
 U 1 1 61748B8C
 P 2800 5800
-F 0 "D70" V 2846 5730 50  0000 R CNN
+F 0 "D61" V 2846 5730 50  0000 R CNN
 F 1 "SOD-123" V 2755 5730 50  0000 R CNN
 F 2 "Diode_SMD:D_SOD-123" V 2800 5800 50  0001 C CNN
@@
 Connection ~ 3850 5900
 Wire Wire Line
-	3850 5900 7400 5900
+	3850 5900 4350 5900
 Wire Wire Line
 	4150 4800 4150 5500
 Connection ~ 4150 4800
-Wire Wire Line
-	4650 4800 4650 5450
 Connection ~ 4650 4800
+Wire Wire Line
+	3050 4350 3050 4550
+Wire Wire Line
+	2950 4150 3150 4150
+Connection ~ 4350 5900
+Wire Wire Line
+	4350 5900 5850 5900
+Wire Wire Line
+	4650 4800 4650 5500
+Connection ~ 5850 5900
+Wire Wire Line
+	5850 5900 7400 5900
+Wire Wire Line
+	6150 4800 6150 5500
+Wire Wire Line
+	13650 3850 14100 3850
+Wire Wire Line
+	13400 4150 13700 4150
 $EndSCHEMATC

Commit message: routing
Parts:
- SW1: footprint random-keyboard-parts:SKQG-1155865 -> Button_Switch_SMD:SW_SPST_SKQG_WithStem
Connections:
- net EncSW is gone; now on net COL8: U2.25 (PD4)
- net COL0: now also U2.22 (PD5)
- net COL1: now also U2.32 (PC7)
- net COL10: now also U2.37 (PF6)
- net COL11: now also U2.38 (PF5)
- net COL12: now also U2.39 (PF4)
- net COL13: now also U2.40 (PF1)
- net COL14: now also U2.41 (PF0)
- net COL2: now also U2.26 (PD6)
- net COL3: now also U2.27 (PD7)
- net COL4: now also U2.28 (PB4)
- net COL5: now also U2.29 (PB5)
- net COL6: now also U2.30 (PB6)
- net COL7: now also U2.31 (PC6)
- net COL9: now also U2.36 (PF7)
- net EncA: now also U2.21 (PD3); no longer U2.22 (PD5)
- net EncB: now also U2.20 (PD2); no longer U2.21 (PD3)
- net GND: now also R6.2; no longer R6.1
- net ROW0: now also U2.12 (PB7)
- net ROW1: now also U2.11 (PB3)
- net ROW2: now also U2.10 (PB2)
- net ROW3: now also U2.9 (PB1)
- net ROW4: now also U2.8 (PB0)
- net at U2.33 (~HWB~/PE2): now also R6.1; no longer R6.2
- net DP: now reaches R1.2, U1.3 (IO2), USB1.5 (DN2), USB1.7 (DN1)
- net DN: now reaches R3.1, U1.2 (IO1), USB1.6 (DP1), USB1.8 (DP2)
- no-connect marks 2 -> 4
Other:
- moved on the sheet: R6
